File: electronics/xboard.sch (EAGLE design)
At the start: 33 parts

Commit message: Buzzer 10mm
Parts:
- BUZZER: value BUZZER66 -> BUZZER10MM; device rhoban:BUZZER66 -> rhoban:BUZZER10MM
Changed lines of the file:
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@@
 <part name="U$12" library="rhoban" deviceset="NPN" device="_BC817,215"/>
 <part name="R8" library="rcl" deviceset="R-EU_" device="R0805" value="470"/>
-<part name="BUZZER" library="rhoban" deviceset="BUZZER" device="66"/>
+<part name="BUZZER" library="rhoban" deviceset="BUZZER" device="10MM"/>
 <part name="GND23" library="supply1" deviceset="GND" device=""/>
 <part name="P+16" library="supply1" deviceset="VCC" device=""/>

Commit message: XBoard
Parts:
- BUZZER: value BUZZER10MM -> BUZZER66; device rhoban:BUZZER10MM -> rhoban:BUZZER66
Changed lines of the file:
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@@
 <part name="U$12" library="rhoban" deviceset="NPN" device="_BC817,215"/>
 <part name="R8" library="rcl" deviceset="R-EU_" device="R0805" value="470"/>
-<part name="BUZZER" library="rhoban" deviceset="BUZZER" device="10MM"/>
+<part name="BUZZER" library="rhoban" deviceset="BUZZER" device="66"/>
 <part name="GND23" library="supply1" deviceset="GND" device=""/>
 <part name="P+16" library="supply1" deviceset="VCC" device=""/>
